File: hardware/alu/alu.kicad_pcb (KiCad board)
At the start: 4 copper layers, 50 x 50 mm, 70 parts, among them J1 Conn_ALU, J2 Conn_Power, U1 74LVC1G02, U10 74AUC2G04, U11 74HC4017, U12 74LVC1G157, U13 74HC595, U14 74HC86, U15 74LVC1G32, U16 74LVC1G08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

Commit message: Unified footprints
Parts:
- U21, U22, U23, U24, U5: footprint Package_TO_SOT_SMD:SOT-23-5 -> Package_TO_SOT_SMD:SOT-23-5_HandSoldering
- moved C23 1.04 mm to (76.8, 114.3)
- moved C22 0.63 mm to (76.2, 110.0), turned to 270 degrees
- moved C21 0.60 mm to (64.8, 101.4)
- moved C24 0.43 mm to (92.0, 81.2)
Routing:
- net /V_IN: track 15.1 -> 12.2 mm
- net /ALU_S0: track 46.1 -> 43.8 mm
- net VCC: track 122.0 -> 122.8 mm, vias 38 -> 36
- net /DBL: track 14.8 -> 15.3 mm
- net GND: track 141.2 -> 141.7 mm, vias 39 -> 41
Other:
- board text added: "2020-06-11"
- board text removed: "2020-05-25"

Commit message: Added placeholders for JLCPCB serial numbers
Other:
- board text added: "JLCJLCJLCJLC"
Changed lines of the file:
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@@
   (general
     (thickness 1.6)
-    (drawings 21)
+    (drawings 22)
     (tracks 1016)
     (zones 0)
@@
     )
   )
+  (gr_text JLCJLCJLCJLC (at 60.25 103 90) (layer F.SilkS)
+    (effects (font (size 1 1) (thickness 0.15)))
+  )
   (gr_text GND (at 99 97.75) (layer B.SilkS)
