File: hardware/alu/alu.kicad_pcb (KiCad board)
At the start: 4 copper layers, 50 x 50 mm, 71 parts, among them J1 Conn_ALU, J2 Conn_Power, U1 74LVC1G02, U10 74AUC2G04, U11 74HC4017, U12 74LVC1G157, U13 74HC595, U14 74HC86, U15 74LVC1G32, U16 74LVC1G08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

Commit message: Update all to Kicad 6
Connections:
- net /A&~B renamed /A&~{B}
- net /B_OR_~B renamed /B_OR_~{B}
- net /EQ_FF_~Q renamed /EQ_FF_~{Q}
- net /~ALU_RESET renamed /~{ALU_RESET}
- net /~A~&B renamed /~{A}&B
- net /~C~_FF_~R~ renamed /~{C}_FF_~{R}
- net /~C~_FF_~S~ renamed /~{C}_FF_~{S}
- net /~OUT_C renamed /~{OUT_C}
- net /~OUT_NEG renamed /~{OUT_NEG}
- net /~SH_OUTPUT renamed /~{SH_OUTPUT}
Other:
- net class Default removed
