File: hardware/power-splitter/power-splitter.kicad_pcb (KiCad board)
At the start: 2 copper layers, 32 x 25 mm, 6 parts, among them J1 Conn_Power, J3 Conn_01x02_Female, J4 Conn_01x02_Female

Commit message: Added placeholders for JLCPCB serial numbers
Other:
- board text added: "JLCJLCJLCJLC"
Changed lines of the file:
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@@
   (general
     (thickness 1.6)
-    (drawings 16)
+    (drawings 17)
     (tracks 39)
     (zones 0)
@@
   )
   (setup
-    (last_trace_width 0.5)
+    (last_trace_width 0.25)
     (user_trace_width 0.5)
     (trace_clearance 0.2)
@@
     )
   )
+  (gr_text JLCJLCJLCJLC (at 67.5 67) (layer B.SilkS)
+    (effects (font (size 1 1) (thickness 0.15)) (justify mirror))
+  )
   (gr_text +5V (at 53.8 58.4) (layer F.SilkS)
