File: hardware/register-bank/register-bank.kicad_pcb (KiCad board)
At the start: 2 copper layers, 51.6 x 51.6 mm, 64 parts, among them J1 Conn_Reg, J2 Conn_Power, U1 HEF4557B, U10 74HC251, U11 74HC251, U12 MIC5504-3.3YM5, U13 74LVC1G04, U14 74LVC1G04, U15 74LVC1G04, U16 74LVC1G04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

Commit message: Unified footprints
Parts:
- U12, U13, U14, U15, U16, U17, U18, U19, U20: footprint Package_TO_SOT_SMD:SOT-23-5 -> Package_TO_SOT_SMD:SOT-23-5_HandSoldering
- moved U17 0.42 mm to (103.2, 114.4)
- moved U18 0.42 mm to (94.6, 114.4)
- moved U19 0.42 mm to (85.7, 114.4)
- moved U20 0.42 mm to (76.8, 114.4)
- moved U15 0.31 mm to (95.6, 72.4)
- moved U13 0.31 mm to (77.8, 72.4)
- moved U14 0.31 mm to (86.7, 72.4)
- moved U16 0.31 mm to (101.6, 72.4)
Routing:
- net GND: track 491.4 -> 500.2 mm
- net VCC: track 293.3 -> 295.8 mm, vias 16 -> 17
Other:
- board text added: "2020-06-11"
- board text removed: "2020-05-27"

Commit message: Added placeholders for JLCPCB serial numbers
Other:
- board text added: "0"
- board text added: "JLCJLCJLCJLC"
Changed lines of the file:
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@@
   (general
     (thickness 1.6)
-    (drawings 17)
+    (drawings 19)
     (tracks 1025)
     (zones 0)
@@
   )
   (setup
-    (last_trace_width 0.5)
+    (last_trace_width 0.25)
     (user_trace_width 0.35)
     (user_trace_width 0.5)
@@
       (xy 0.1016 -0.166391)) (layer B.SilkS) (width 0.01))
   )
+  (gr_text 0 (at 78.9 80.645) (layer F.SilkS)
+    (effects (font (size 1.5 1.5) (thickness 0.3)))
+  )
+  (gr_text JLCJLCJLCJLC (at 64.25 93 90) (layer F.SilkS)
+    (effects (font (size 1 1) (thickness 0.15)))
+  )
   (gr_text GND (at 111.75 104.25 270) (layer B.SilkS)
