File: hardware/register-bank/register-bank.sch (KiCad schematic (older format))
At the start: 62 parts, among them J1 Conn_Reg, J2 Conn_Power, U1 HEF4557B, U10 74HC251, U11 74HC251, U12 MIC5504-3.3YM5, U13 74LVC1G04, U14 74LVC1G04, U15 74LVC1G04, U16 74LVC1G04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

Commit message: Unified footprints
Parts:
- U12, U13, U14, U15, U16, U17, U18, U19, U20: footprint Package_TO_SOT_SMD:SOT-23-5 -> Package_TO_SOT_SMD:SOT-23-5_HandSoldering
Changed lines of the file:
@@
 F 0 "U12" H 4400 9867 50  0000 C CNN
 F 1 "MIC5504-3.3YM5" H 4400 9776 50  0000 C CNN
-F 2 "Package_TO_SOT_SMD:SOT-23-5" H 4400 9100 50  0001 C CNN
+F 2 "Package_TO_SOT_SMD:SOT-23-5_HandSoldering" H 4400 9100 50  0001 C CNN
 F 3 "http://ww1.microchip.com/downloads/en/DeviceDoc/MIC550X.pdf" H 4150 9750 50  0001 C CNN
 	1    4400 9500
@@
 F 0 "U13" H 10300 4800 50  0000 C CNN
 F 1 "74LVC1G04" H 10300 5176 50  0000 C CNN
-F 2 "Package_TO_SOT_SMD:SOT-23-5" H 10300 5000 50  0001 C CNN
+F 2 "Package_TO_SOT_SMD:SOT-23-5_HandSoldering" H 10300 5000 50  0001 C CNN
 F 3 "" H 10300 5000 50  0001 C CNN
 	1    10300 5000
@@
 F 0 "U13" H 5880 10096 50  0000 L CNN
 F 1 "74LVC1G04" H 5880 10005 50  0000 L CNN
-F 2 "Package_TO_SOT_SMD:SOT-23-5" H 5750 10050 50  0001 C CNN
+F 2 "Package_TO_SOT_SMD:SOT-23-5_HandSoldering" H 5750 10050 50  0001 C CNN
 F 3 "" H 5750 10050 50  0001 C CNN
 	2    5750 10050
@@
 F 0 "U14" H 10300 5300 50  0000 C CNN
 F 1 "74LVC1G04" H 10300 5676 50  0000 C CNN
-F 2 "Package_TO_SOT_SMD:SOT-23-5" H 10300 5500 50  0001 C CNN
+F 2 "Package_TO_SOT_SMD:SOT-23-5_HandSoldering" H 10300 5500 50  0001 C CNN
 F 3 "" H 10300 5500 50  0001 C CNN
 	1    10300 5500
@@
 F 0 "U15" H 10300 5800 50  0000 C CNN
 F 1 "74LVC1G04" H 10300 6176 50  0000 C CNN
-F 2 "Package_TO_SOT_SMD:SOT-23-5" H 10300 6000 50  0001 C CNN
+F 2 "Package_TO_SOT_SMD:SOT-23-5_HandSoldering" H 10300 6000 50  0001 C CNN
 F 3 "" H 10300 6000 50  0001 C CNN
 	1    10300 6000
@@
 F 0 "U16" H 10300 6300 50  0000 C CNN
 F 1 "74LVC1G04" H 10300 6676 50  0000 C CNN
-F 2 "Package_TO_SOT_SMD:SOT-23-5" H 10300 6500 50  0001 C CNN
+F 2 "Package_TO_SOT_SMD:SOT-23-5_HandSoldering" H 10300 6500 50  0001 C CNN
 F 3 "" H 10300 6500 50  0001 C CNN
 	1    10300 6500
@@
 F 0 "U17" H 10300 6800 50  0000 C CNN
 F 1 "74LVC1G04" H 10300 7176 50  0000 C CNN
-F 2 "Package_TO_SOT_SMD:SOT-23-5" H 10300 7000 50  0001 C CNN
+F 2 "Package_TO_SOT_SMD:SOT-23-5_HandSoldering" H 10300 7000 50  0001 C CNN
 F 3 "" H 10300 7000 50  0001 C CNN
 	1    10300 7000
@@
 F 0 "U18" H 10300 7300 50  0000 C CNN
 F 1 "74LVC1G04" H 10300 7676 50  0000 C CNN
-F 2 "Package_TO_SOT_SMD:SOT-23-5" H 10300 7500 50  0001 C CNN
+F 2 "Package_TO_SOT_SMD:SOT-23-5_HandSoldering" H 10300 7500 50  0001 C CNN
 F 3 "" H 10300 7500 50  0001 C CNN
 	1    10300 7500
@@
 F 0 "U19" H 10300 7800 50  0000 C CNN
 F 1 "74LVC1G04" H 10300 8176 50  0000 C CNN
-F 2 "Package_TO_SOT_SMD:SOT-23-5" H 10300 8000 50  0001 C CNN
+F 2 "Package_TO_SOT_SMD:SOT-23-5_HandSoldering" H 10300 8000 50  0001 C CNN
 F 3 "" H 10300 8000 50  0001 C CNN
 	1    10300 8000
@@
 F 0 "U20" H 10300 8300 50  0000 C CNN
 F 1 "74LVC1G04" H 10300 8676 50  0000 C CNN
-F 2 "Package_TO_SOT_SMD:SOT-23-5" H 10300 8500 50  0001 C CNN
+F 2 "Package_TO_SOT_SMD:SOT-23-5_HandSoldering" H 10300 8500 50  0001 C CNN
 F 3 "" H 10300 8500 50  0001 C CNN
 	1    10300 8500
@@
 F 0 "U14" H 6630 10096 50  0000 L CNN
 F 1 "74LVC1G04" H 6630 10005 50  0000 L CNN
-F 2 "Package_TO_SOT_SMD:SOT-23-5" H 6500 10050 50  0001 C CNN
+F 2 "Package_TO_SOT_SMD:SOT-23-5_HandSoldering" H 6500 10050 50  0001 C CNN
 F 3 "" H 6500 10050 50  0001 C CNN
 	2    6500 10050
@@
 F 0 "U15" H 7380 10096 50  0000 L CNN
 F 1 "74LVC1G04" H 7380 10005 50  0000 L CNN
-F 2 "Package_TO_SOT_SMD:SOT-23-5" H 7250 10050 50  0001 C CNN
+F 2 "Package_TO_SOT_SMD:SOT-23-5_HandSoldering" H 7250 10050 50  0001 C CNN
 F 3 "" H 7250 10050 50  0001 C CNN
 	2    7250 10050
@@
 F 0 "U16" H 8130 10096 50  0000 L CNN
 F 1 "74LVC1G04" H 8130 10005 50  0000 L CNN
-F 2 "Package_TO_SOT_SMD:SOT-23-5" H 8000 10050 50  0001 C CNN
+F 2 "Package_TO_SOT_SMD:SOT-23-5_HandSoldering" H 8000 10050 50  0001 C CNN
 F 3 "" H 8000 10050 50  0001 C CNN
 	2    8000 10050
@@
 F 0 "U17" H 8880 10096 50  0000 L CNN
 F 1 "74LVC1G04" H 8880 10005 50  0000 L CNN
-F 2 "Package_TO_SOT_SMD:SOT-23-5" H 8750 10050 50  0001 C CNN
+F 2 "Package_TO_SOT_SMD:SOT-23-5_HandSoldering" H 8750 10050 50  0001 C CNN
 F 3 "" H 8750 10050 50  0001 C CNN
 	2    8750 10050
@@
 F 0 "U18" H 9630 10096 50  0000 L CNN
 F 1 "74LVC1G04" H 9630 10005 50  0000 L CNN
-F 2 "Package_TO_SOT_SMD:SOT-23-5" H 9500 10050 50  0001 C CNN
+F 2 "Package_TO_SOT_SMD:SOT-23-5_HandSoldering" H 9500 10050 50  0001 C CNN
 F 3 "" H 9500 10050 50  0001 C CNN
 	2    9500 10050
@@
 F 0 "U19" H 10380 10096 50  0000 L CNN
 F 1 "74LVC1G04" H 10380 10005 50  0000 L CNN
-F 2 "Package_TO_SOT_SMD:SOT-23-5" H 10250 10050 50  0001 C CNN
+F 2 "Package_TO_SOT_SMD:SOT-23-5_HandSoldering" H 10250 10050 50  0001 C CNN
 F 3 "" H 10250 10050 50  0001 C CNN
 	2    10250 10050
@@
 F 0 "U20" H 11130 10096 50  0000 L CNN
 F 1 "74LVC1G04" H 11130 10005 50  0000 L CNN
-F 2 "Package_TO_SOT_SMD:SOT-23-5" H 11000 10050 50  0001 C CNN
+F 2 "Package_TO_SOT_SMD:SOT-23-5_HandSoldering" H 11000 10050 50  0001 C CNN
 F 3 "" H 11000 10050 50  0001 C CNN
 	2    11000 10050

Commit message: Added test points
Parts:
- added TP1: TestPoint, TestPoint:TestPoint_THTPad_D2.0mm_Drill1.0mm, symbol Connector:TestPoint
Connections:
- net GND: now also TP1.1

Commit message: Update all to Kicad 6
Connections:
- net ~RIN_EN renamed ~{RIN_EN}
- net ~RIN_EN0 renamed ~{RIN_EN0}
- net ~RIN_EN1 renamed ~{RIN_EN1}
- net ~RIN_EN2 renamed ~{RIN_EN2}
- net ~RIN_EN3 renamed ~{RIN_EN3}
- net ~RIN_EN4 renamed ~{RIN_EN4}
- net ~RIN_EN5 renamed ~{RIN_EN5}
- net ~RIN_EN6 renamed ~{RIN_EN6}
- net ~RIN_EN7 renamed ~{RIN_EN7}
- net ~ROUT_EN_A renamed ~{ROUT_EN_A}
- net ~ROUT_EN_B renamed ~{ROUT_EN_B}
