File: hardware/memory-io/memory-io.kicad_pcb (KiCad board)
At the start: 4 copper layers, 134.8 x 246.8 mm, 172 parts, among them J1 Conn_Mem_Ext, J2 Conn_Power, J3 DOGM162S-A, J4 SD_Card, J5 Conn_01x03_Male, J6 FTDI, SW1 SW_Push_4pin, SW2 SW_Push_4pin, SW3 SW_Push_4pin, SW4 SW_Push_4pin, SW5 SW_Push_4pin, SW6 SW_Push_4pin, SW7 SW_Push_4pin, U1 74HC74, U10 74HC688, U11 74LVC1G38, U12 74LVC1G38, U13 74LVC1G04, U14 74HC541, U15 74LVC1G32, U16 74LVC1G08, U17 74LVC2G74, U18 74HC273, U19 74HC597, U2 74HC139, U20 74LVC1G04, U22 74LVC2G74, U23 74LVC1G04, U24 SC16C550B, U25 74HC574, U26 74HC597, U27 74HC595, U28 74LVC1G04, U29 74HC9115, U3 74LVC1G08, U30 74LVC1G04, U31 74LVC2G74, U4 74LVC1G04, U5 74HC02, U6 74HC32, U7 74LVC1G14, U8 MCP1825S, U9 74HC138, Y1 1.8432MHz

Commit message: Update all to Kicad 6
Connections:
- net /~LCD_E renamed /~{LCD_E}
- net /~LED_E renamed /~{LED_E}
- net /~MEM_OE renamed /~{MEM_OE}
- net /~MEM_WE renamed /~{MEM_WE}
- net /~RESET renamed /~{RESET}
- net /~SD_CS renamed /~{SD_CS}
- net /~SD_DATA_OE renamed /~{SD_DATA_OE}
- net /~SD_DATA_OE_IN renamed /~{SD_DATA_OE_IN}
- net /~SD_DATA_TRIG renamed /~{SD_DATA_TRIG}
- net /~SD_DATA_WE renamed /~{SD_DATA_WE}
- net /~SD_DATA_WE_IN renamed /~{SD_DATA_WE_IN}
- net /~SD_DUMMY_READ renamed /~{SD_DUMMY_READ}
- net /~SD_E renamed /~{SD_E}
- net /~SD_SCLK renamed /~{SD_SCLK}
- net /~SD_SPI_EN renamed /~{SD_SPI_EN}
- net /~SD_STATUS_OE renamed /~{SD_STATUS_OE}
- net /~SD_STATUS_WE renamed /~{SD_STATUS_WE}
- net /~SWITCH_E renamed /~{SWITCH_E}
- net /~SWITCH_OE renamed /~{SWITCH_OE}
- net /~SW_ANY renamed /~{SW_ANY}
- net /~SW_IRQ renamed /~{SW_IRQ}
- net /~SW_RESET renamed /~{SW_RESET}
- net /~UART_E renamed /~{UART_E}
- net /~UART_IRQ renamed /~{UART_IRQ}
- net /~WAIT renamed /~{WAIT}
Other:
- net class Default removed
