File: hardware/memory-ram/memory-ram.kicad_pcb (KiCad board)
At the start: 2 copper layers, 77 x 39 mm, 27 parts, among them J1 Conn_Mem_Ext, J2 Conn_Power, U1 IS61WV5128EDBLL-10TLI, U2 74LVC1G86, U3 MIC5504-3.3YM5, U4 74LVC1G32, U5 74LVC1G332, U6 74LVC1G86, U7 74LVC1G04

Commit message: Added test points
Parts:
- added TP1: TestPoint, TestPoint:TestPoint_THTPad_D2.0mm_Drill1.0mm, F.Cu at (84.6, 98.0)
Routing:
- net GND: track 171.9 -> 201.5 mm
Changed lines of the file:
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@@
     (thickness 1.6)
     (drawings 19)
-    (tracks 513)
+    (tracks 516)
     (zones 0)
-    (modules 27)
+    (modules 28)
     (nets 62)
   )
@@
   )
   (setup
-    (last_trace_width 0.25)
+    (last_trace_width 0.35)
     (user_trace_width 0.35)
     (user_trace_width 0.5)
@@
       (rotate (xyz -90 0 0))
     )
+  )
+  (module TestPoint:TestPoint_THTPad_D2.0mm_Drill1.0mm (layer F.Cu)
+    (at 84.6 98)
+    (descr "THT pad as test Point, diameter 2.0mm, hole diameter 1.0mm")
+    (tags "test point THT pad")
+    (attr virtual)
+    (fp_text reference TP1 (at 0 -1.998) (layer F.SilkS) hide
+      (effects (font (size 1 1) (thickness 0.15)))
+    )
+    (fp_text value TestPoint (at 0 2.05) (layer F.Fab)
+      (effects (font (size 1 1) (thickness 0.15)))
+    )
+    (fp_text user %R (at 0 -2) (layer F.Fab)
+      (effects (font (size 1 1) (thickness 0.15)))
+    )
+    (fp_circle (center 0 0) (end 1.5 0) (layer F.CrtYd) (width 0.05))
+    (fp_circle (center 0 0) (end 0 1.2) (layer F.SilkS) (width 0.12))
+    (pad 1 thru_hole circle (at 0 0) (size 2 2) (drill 1) (layers *.Cu *.Mask)
+      (net 9 GND))
   )
   (gr_text JLCJLCJLCJLC (at 101.525 129.375) (layer F.SilkS)
@@
   (segment (start 96.325 114.75) (end 96.975 114.75) (width 0.35) (layer B.Cu) (net 9))
   (segment (start 96.975 114.75) (end 99.45 114.75) (width 0.35) (layer B.Cu) (net 9))
+  (segment (start 84.6 98) (end 87 100.4) (width 0.35) (layer B.Cu) (net 9))
+  (segment (start 108.3 100.4) (end 111.7 103.8) (width 0.35) (layer B.Cu) (net 9))
+  (segment (start 87 100.4) (end 108.3 100.4) (width 0.35) (layer B.Cu) (net 9))
   (segment (start 119.176101 129.376101) (end 119.176101 125.648601) (width 0.25) (layer F.Cu) (net 10))
   (segment (start 125.8 115.6) (end 130 119.8) (width 0.25) (layer F.Cu) (net 10))

Commit message: Update all to Kicad 6
Connections:
- net /~A31 renamed /~{A31}
- net /~CE renamed /~{CE}
- net /~MEM_OE renamed /~{MEM_OE}
- net /~MEM_WE renamed /~{MEM_WE}
- net /~RESET renamed /~{RESET}
- net /~WAIT renamed /~{WAIT}
Other:
- net class Default removed
