File: hardware/pc/pc.kicad_pcb (KiCad board)
At the start: 2 copper layers, 68 x 100 mm, 128 parts, among them J1 Conn_Power, J2 Conn_PC, U1 74HC161, U10 74HC597, U11 74HC595, U12 74HC161, U13 74HC161, U14 74HC597, U15 74HC595, U16 74HC161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

Commit message: Added test points
Parts:
- added TP1: TestPoint, TestPoint:TestPoint_THTPad_D2.0mm_Drill1.0mm, F.Cu at (155.8, 137.4)
Changed lines of the file:
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@@
     (tracks 1844)
     (zones 0)
-    (modules 128)
+    (modules 129)
     (nets 166)
   )
@@
       (xy 0.1016 -0.166391)) (layer B.SilkS) (width 0.01))
   )
+  (module TestPoint:TestPoint_THTPad_D2.0mm_Drill1.0mm (layer F.Cu)
+    (at 155.8 137.4)
+    (descr "THT pad as test Point, diameter 2.0mm, hole diameter 1.0mm")
+    (tags "test point THT pad")
+    (attr virtual)
+    (fp_text reference TP1 (at 0 -1.998) (layer F.SilkS) hide
+      (effects (font (size 1 1) (thickness 0.15)))
+    )
+    (fp_text value TestPoint (at 0 2.05) (layer F.Fab)
+      (effects (font (size 1 1) (thickness 0.15)))
+    )
+    (fp_text user %R (at 0 -2) (layer F.Fab)
+      (effects (font (size 1 1) (thickness 0.15)))
+    )
+    (fp_circle (center 0 0) (end 1.5 0) (layer F.CrtYd) (width 0.05))
+    (fp_circle (center 0 0) (end 0 1.2) (layer F.SilkS) (width 0.12))
+    (pad 1 thru_hole circle (at 0 0) (size 2 2) (drill 1) (layers *.Cu *.Mask)
+      (net 2 GND))
+  )
   (gr_text +5V (at 149.5 70.5) (layer B.SilkS)

Commit message: Update all to Kicad 6
Connections:
- net /CNT_~PE renamed /CNT_~{PE}
- net /OUT_S~P~ renamed /OUT_S~{P}
- net /Q1_OR_~Q1 renamed /Q1_OR_~{Q1}
- net /~Q1 renamed /~{Q1}
- net /~RESET renamed /~{RESET}
Other:
- net class Default removed
