File: hardware/test-bench/test-bench.kicad_pcb (KiCad board)
At the start: 2 copper layers, 90 x 90 mm, 46 parts, among them J1 Conn_Mem_Ext, J2 Conn_Reg, J3 SWD, J4 Conn_Mem, J5 FTDI, J6 Conn_Power, J7 J_LINK_SWD, SW1 SW_Push_4pin, SW2 SW_Push_4pin, U1 STM32G030F6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

Commit message: Update all to Kicad 6
Connections:
- net /~CS renamed /~{CS}
- net /~RESET renamed /~{RESET}
Other:
- net class Default removed
- board text added: "~{RESET}"
- board text removed: "~RESET"
