File: hardware/opcode/Imm24.kicad_sch (KiCad schematic)
At the start: 6 parts, among them U20 74HC597, U21 74HC597, U22 74HC597

Commit message: Update all to Kicad 6
Parts:
- renumbered C4 to C6, C5 to C7, C6 to C8, U20 to U25, U21 to U26, U22 to U27
Changed lines of the file:
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@@
   (symbol (lib_id "riscv-serial:74HC597") (at 74.93 142.24 0) (unit 1)
     (in_bom yes) (on_board yes)
-    (property "Reference" "U21" (id 0) (at 78.74 163.83 0)
+    (property "Reference" "U26" (id 0) (at 78.74 163.83 0)
       (effects (font (size 1.27 1.27)) (justify left))
     )
@@
   (symbol (lib_id "power:VCC") (at 74.93 114.3 0) (unit 1)
     (in_bom yes) (on_board yes)
-    (property "Reference" "#PWR0145" (id 0) (at 74.93 118.11 0)
+    (property "Reference" "#PWR059" (id 0) (at 74.93 118.11 0)
       (effects (font (size 1.27 1.27)) hide)
     )
@@
   (symbol (lib_id "Device:C") (at 93.98 118.11 0) (unit 1)
     (in_bom yes) (on_board yes)
-    (property "Reference" "C5" (id 0) (at 96.901 116.9416 0)
+    (property "Reference" "C7" (id 0) (at 96.901 116.9416 0)
       (effects (font (size 1.27 1.27)) (justify left))
     )
@@
   (symbol (lib_id "power:VCC") (at 74.93 182.88 0) (unit 1)
     (in_bom yes) (on_board yes)
-    (property "Reference" "#PWR0149" (id 0) (at 74.93 186.69 0)
+    (property "Reference" "#PWR063" (id 0) (at 74.93 186.69 0)
       (effects (font (size 1.27 1.27)) hide)
     )
@@
   (symbol (lib_id "power:GND") (at 74.93 234.95 0) (unit 1)
     (in_bom yes) (on_board yes)
-    (property "Reference" "#PWR0150" (id 0) (at 74.93 241.3 0)
+    (property "Reference" "#PWR065" (id 0) (at 74.93 241.3 0)
       (effects (font (size 1.27 1.27)) hide)
     )
@@
   (symbol (lib_id "Device:C") (at 93.98 186.69 0) (unit 1)
     (in_bom yes) (on_board yes)
-    (property "Reference" "C6" (id 0) (at 96.901 185.5216 0)
+    (property "Reference" "C8" (id 0) (at 96.901 185.5216 0)
       (effects (font (size 1.27 1.27)) (justify left))
     )
@@
   (symbol (lib_id "power:VCC") (at 93.98 181.61 0) (unit 1)
     (in_bom yes) (on_board yes)
-    (property "Reference" "#PWR0151" (id 0) (at 93.98 185.42 0)
+    (property "Reference" "#PWR062" (id 0) (at 93.98 185.42 0)
       (effects (font (size 1.27 1.27)) hide)
     )
@@
   (symbol (lib_id "riscv-serial:74HC597") (at 74.93 73.66 0) (unit 1)
     (in_bom yes) (on_board yes)
-    (property "Reference" "U20" (id 0) (at 78.74 95.25 0)
+    (property "Reference" "U25" (id 0) (at 78.74 95.25 0)
       (effects (font (size 1.27 1.27)) (justify left))
     )
@@
   (symbol (lib_id "power:VCC") (at 74.93 45.72 0) (unit 1)
     (in_bom yes) (on_board yes)
-    (property "Reference" "#PWR0153" (id 0) (at 74.93 49.53 0)
+    (property "Reference" "#PWR055" (id 0) (at 74.93 49.53 0)
       (effects (font (size 1.27 1.27)) hide)
     )
@@
   (symbol (lib_id "Device:C") (at 93.98 49.53 0) (unit 1)
     (in_bom yes) (on_board yes)
-    (property "Reference" "C4" (id 0) (at 96.901 48.3616 0)
+    (property "Reference" "C6" (id 0) (at 96.901 48.3616 0)
       (effects (font (size 1.27 1.27)) (justify left))
     )
@@
   (symbol (lib_id "power:VCC") (at 93.98 44.45 0) (unit 1)
     (in_bom yes) (on_board yes)
-    (property "Reference" "#PWR0155" (id 0) (at 93.98 48.26 0)
+    (property "Reference" "#PWR054" (id 0) (at 93.98 48.26 0)
       (effects (font (size 1.27 1.27)) hide)
     )
@@
   (symbol (lib_id "power:GND") (at 93.98 54.61 0) (unit 1)
     (in_bom yes) (on_board yes)
-    (property "Reference" "#PWR0156" (id 0) (at 93.98 60.96 0)
+    (property "Reference" "#PWR056" (id 0) (at 93.98 60.96 0)
       (effects (font (size 1.27 1.27)) hide)
     )
@@
   (symbol (lib_id "power:VCC") (at 93.98 113.03 0) (unit 1)
     (in_bom yes) (on_board yes)
-    (property "Reference" "#PWR0147" (id 0) (at 93.98 116.84 0)
+    (property "Reference" "#PWR058" (id 0) (at 93.98 116.84 0)
       (effects (font (size 1.27 1.27)) hide)
     )
@@
   (symbol (lib_id "power:GND") (at 93.98 123.19 0) (unit 1)
     (in_bom yes) (on_board yes)
-    (property "Reference" "#PWR0148" (id 0) (at 93.98 129.54 0)
+    (property "Reference" "#PWR060" (id 0) (at 93.98 129.54 0)
       (effects (font (size 1.27 1.27)) hide)
     )
@@
   (symbol (lib_id "riscv-serial:74HC597") (at 74.93 210.82 0) (unit 1)
     (in_bom yes) (on_board yes)
-    (property "Reference" "U22" (id 0) (at 78.74 232.41 0)
+    (property "Reference" "U27" (id 0) (at 78.74 232.41 0)
       (effects (font (size 1.27 1.27)) (justify left))
     )
@@
   (symbol (lib_id "power:GND") (at 74.93 97.79 0) (unit 1)
     (in_bom yes) (on_board yes)
-    (property "Reference" "#PWR0154" (id 0) (at 74.93 104.14 0)
+    (property "Reference" "#PWR057" (id 0) (at 74.93 104.14 0)
       (effects (font (size 1.27 1.27)) hide)
     )
@@
   (symbol (lib_id "power:GND") (at 74.93 166.37 0) (unit 1)
     (in_bom yes) (on_board yes)
-    (property "Reference" "#PWR0146" (id 0) (at 74.93 172.72 0)
+    (property "Reference" "#PWR061" (id 0) (at 74.93 172.72 0)
       (effects (font (size 1.27 1.27)) hide)
     )
@@
   (symbol (lib_id "power:GND") (at 93.98 191.77 0) (unit 1)
     (in_bom yes) (on_board yes)
-    (property "Reference" "#PWR0152" (id 0) (at 93.98 198.12 0)
-      (effects (font (size 1.27 1.27)) hide)
-    )
+    (property "Reference" "#PWR064" (id 0) (at 93.98 198.12 0)
+      (effects (font (size 1.27 1.27)) hide)
+    )
