File: hardware/opcode/opcode.kicad_sch (KiCad schematic)
At the start: 36 parts, among them J1 Conn_01x40, J2 Conn_01x14, J3 Conn_01x20, U1 74HC595, U10 74LVC1G32, U11 74LVC1G32, U12 SST39SF040, U13 SST39SF040, U14 SST39SF040, U15 SST39SF040, U16 74HC251, U2 74HC595, U3 74HC595, U31 74LVC1G08, U4 74HC595, U5 74LVC1G00, U6 74LVC1G08, U7 74HC595, U8 74HC74, U9 74LVC1G00

Commit message: Update all to Kicad 6
Parts:
- added U13, U19: 74LVC1G32, Package_TO_SOT_SMD:SOT-23-5_HandSoldering, symbol riscv-serial:74LVC1G32
- U17: renamed from U31; footprint (none) -> Package_TO_SOT_SMD:SOT-23-5_HandSoldering
- renumbered U8 to U1, U5 to U10, U3 to U11, U6 to U12, U4 to U14, U11 to U15, U10 to U16, U16 to U18, U1 to U2, U12 to U3, U13 to U4, U14 to U5, U15 to U6, U2 to U7, U7 to U8
Connections:
- net COMPR: now also U13.2; no longer U2.13 (~{OE}), U7.13 (~{OE})
- net ~{OE}: now also U13.1
- new net COMPR_~{OE}: U13.4, U2.13 (~{OE}), U7.13 (~{OE})
Other:
- moved on the sheet: R1, R10, R11, R12, R13, R14, R15, R16, R2, R3, R4, R5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

Commit message: Updated schematics and pcbs
Parts:
- removed J3: Conn_01x20, Connector_IDC:IDC-Header_2x10_P2.54mm_Vertical, symbol Connector_Generic:Conn_01x20
- removed R1, R10, R11, R12, R13, R14, R15, R16, R2, R3, R4, R5, R6, R7, R8, R9: 10k, Resistor_SMD:R_0805_2012Metric_Pad1.20x1.40mm_HandSolder, symbol Device:R
- added J3: Conn_Reg_Sel, Connector_IDC:IDC-Header_2x10_P2.54mm_Vertical, symbol riscv-serial:Conn_Reg_Sel
- added R1, R10, R11, R12, R13, R14, R15, R16, R17, R18, R19, R2, R20, R21, R22, R23, R24, R25, R26, R27, R28, R29, R3, R30, R31, R32, R4, R5, R6, R7, R8, R9: 10k, riscv-serial:Jumper_3_R_0805, symbol riscv-serial:Jumper_3_R
Connections:
- net A0: now also R1.2
- net A1: now also R2.2
- net A10: now also R11.2
- net A11: now also R12.2
- net A12: now also R13.2
- net A13: now also R14.2
- net A14: now also R15.2
- net A15: now also R16.2
- net A2: now also R3.2
- net A3: now also R4.2
- net A4: now also R5.2
- net A5: now also R6.2
- net A6: now also R7.2
- net A7: now also R8.2
- net A8: now also R9.2
- net A9: now also R10.2
- net B16: now also R17.2
- net B17: now also R18.2
- net B18: now also R19.2
- net B19: now also R20.2
- net B20: now also R21.2
- net B21: now also R22.2
- net B22: now also R23.2
- net B23: now also R24.2
- net B24: now also R25.2
- net B25: now also R26.2
- net B26: now also R27.2
- net B27: now also R28.2
- net B28: now also R29.2
- net B29: now also R30.2
- net B30: now also R31.2
- net B31: now also R32.2
- net GND: now also J3.1 (GND), J3.14 (GND), J3.2 (GND), J3.20 (GND), J3.8 (GND), R1.3, R10.1, R11.1, R12.1, R13.1, R14.1, R15.1, R16.1, R17.1, R18.1, R19.1, R2.3, R20.1, R21.1, R22.1, R23.1, R24.1, R25.1, R26.1, R27.1, R28.1, R29.1, R3.3, R30.1, R31.1, R32.1, R4.1, R5.1, R6.3, R7.3, R8.1, R9.1
- net RAS0: now also J3.15 (RAS0)
- net RAS1: now also J3.16 (RAS1)
- net RAS2: now also J3.17 (RAS2)
- net RAS3: now also J3.18 (RAS3)
- net RAS4: now also J3.19 (RAS4)
- net RBS0: now also J3.9 (RBS0)
- net RBS1: now also J3.10 (RBS1)
- net RBS2: now also J3.11 (RBS2)
- net RBS3: now also J3.12 (RBS3)
- net RBS4: now also J3.13 (RBS4)
- net RINS0: now also J3.3 (RINS0)
- net RINS1: now also J3.4 (RINS1)
- net RINS2: now also J3.5 (RINS2)
- net RINS3: now also J3.6 (RINS3)
- net RINS4: now also J3.7 (RINS4)
- net VCC: now also R1.1, R10.3, R11.3, R12.3, R13.3, R14.3, R15.3, R16.3, R17.3, R18.3, R19.3, R2.1, R20.3, R21.3, R22.3, R23.3, R24.3, R25.3, R26.3, R27.3, R28.3, R29.3, R3.1, R30.3, R31.3, R32.3, R4.3, R5.3, R6.1, R7.1, R8.3, R9.3
Other:
- note added: "Inital instruction: 00000067 jalr x0, 0(x0)"
- note removed: "Inital instruction: A001 c.j 0"

Commit message: Added start of adapter circuits
Parts:
- removed J2: Conn_01x14, symbol Connector_Generic:Conn_01x14
- removed U18: 74HC251, Package_SO:SOIC-16_3.9x9.9mm_P1.27mm, symbol riscv-serial:74HC251
- added J2: Conn_01x24, Connector_IDC:IDC-Header_2x12_P2.54mm_Vertical, symbol Connector_Generic:Conn_01x24
- J1: footprint (none) -> Connector_IDC:IDC-Header_2x20_P2.54mm_Vertical
Connections:
- net ALU_SA: now also J2.12 (Pin_12)
- net B10: now also J1.36 (Pin_36)
- net B11: now also J1.35 (Pin_35)
- net B12: now also J1.34 (Pin_34)
- net B13: now also J1.33 (Pin_33)
- net B14: now also J1.32 (Pin_32)
- net B15: now also J1.31 (Pin_31)
- net B16: now also J1.30 (Pin_30)
- net B17: now also J1.29 (Pin_29)
- net B18: now also J1.28 (Pin_28)
- net B19: now also J1.27 (Pin_27)
- net B20: now also J1.26 (Pin_26)
- net B21: now also J1.25 (Pin_25)
- net B22: now also J1.24 (Pin_24)
- net B23: now also J1.23 (Pin_23)
- net B24: now also J1.22 (Pin_22)
- net B25: now also J1.21 (Pin_21)
- net B26: now also J1.20 (Pin_20)
- net B27: now also J1.19 (Pin_19)
- net B28: now also J1.18 (Pin_18)
- net B29: now also J1.17 (Pin_17)
- net B30: now also J1.16 (Pin_16)
- net B31: now also J1.15 (Pin_15)
- net B7: now also J1.39 (Pin_39)
- net B8: now also J1.38 (Pin_38)
- net B9: now also J1.37 (Pin_37)
- net BUS_CLK: now also J1.2 (Pin_2), J2.2 (Pin_2)
- net GND: now also J1.1 (Pin_1), J1.40 (Pin_40)
- net IMM_LATCH: now also J1.5 (Pin_5), J2.6 (Pin_6)
- net IMM_MUX0: now also J2.8 (Pin_8)
- net IMM_MUX1: now also J2.9 (Pin_9)
- net IMM_MUX2: now also J2.10 (Pin_10)
- net IMM_S~{P}: now also J1.6 (Pin_6), J2.7 (Pin_7)
- net Imm: now also J1.11 (Pin_11)
- net OP_LATCH: now also J2.4 (Pin_4)
- net OP_LATCH_LSB: now also J2.5 (Pin_5)
- net SYS: now also J2.11 (Pin_11)
- net ~{RESET}: now also J1.4 (Pin_4), J2.3 (Pin_3)
- no-connect marks 11 -> 10
Other:
- removed sheet ImmB
- removed sheet ImmCSR
- removed sheet ImmI
- removed sheet ImmJ
- removed sheet ImmS
- removed sheet ImmU
