File: hardware/registers/registers.kicad_pcb (KiCad board)
At the start: 4 copper layers, 101.6 x 44.4 mm, 41 parts, among them J1 Conn_Reg, J2 Conn_Reg, J3 Conn_01x20, J4 Conn_Power, J5 Conn_01x10, J6 Conn_01x10, U1 74LVC1G19, U2 74LVC1G19, U3 74LVC1G19, U4 74LVC1G86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

Commit message: Updated schematics and pcbs
Parts:
- added C10: 100n, Capacitor_SMD:C_0805_2012Metric_Pad1.18x1.45mm_HandSolder, F.Cu at (145.4, 92.7)
- added U9: 74LVC1G04, Package_TO_SOT_SMD:SOT-23-5_HandSoldering, F.Cu at (142.2, 92.7)
- J3: value Conn_01x20 -> Conn_Reg_Sel
- J5, J6: value Conn_01x10 -> Conn_Reg_Data
- moved R3 19.2 mm to (134.9, 94.0), turned to 0 degrees
- moved R5 3.20 mm to (170.2, 88.6)
- moved R6 2.62 mm to (175.5, 92.1)
- moved D3 2.54 mm to (129.5, 94.0)
- moved D4 2.54 mm to (163.8, 94.0)
- moved D2 2.54 mm to (125.7, 94.0)
- moved J5 2.54 mm to (101.0, 77.5)
- moved J6 2.54 mm to (189.9, 77.5)
- moved D1 2.54 mm to (121.9, 94.0)
- moved D5 2.54 mm to (167.6, 94.0)
- moved D6 2.54 mm to (171.4, 94.0)
- moved R4 1.29 mm to (167.9, 86.4)
Connections:
- J5 pad 4: /RESET -> /~{RESET}
- J6 pad 4: /RESET -> /~{RESET}
Routing:
- net /~{RESET}: track 0.00 -> 104.6 mm, vias 0 -> 2
- net /RESET: track 109.8 -> 61.4 mm, vias 1 -> 2
- net Net-(D3-Pad2): track 19.0 -> 4.76 mm
- net VCC: track 210.1 -> 219.5 mm
- net /RAOUT: track 112.5 -> 118.1 mm
- net /RBOUT: track 117.6 -> 123.2 mm
- net /BUS_CLK: track 115.9 -> 120.9 mm
- net /RIN: track 114.9 -> 120.0 mm
- net /~{IN_EN}: track 116.5 -> 120.1 mm
- net GND: track 73.8 -> 76.8 mm, vias 13 -> 15
- net Net-(D2-Pad2): track 12.3 -> 9.74 mm
- net Net-(D1-Pad2): track 7.42 -> 4.88 mm
- net Net-(D5-Pad1): track 8.04 -> 5.55 mm
- net /~{IN_EN_1}: track 46.4 -> 44.0 mm
- net Net-(D4-Pad1): track 10.4 -> 8.77 mm
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