File: hardware/clock/clock.kicad_sch (KiCad schematic)
At the start: 110 parts, among them J1 Conn_Power, J2 Conn_01x04_Female, SW1 SW_Push_4pin, SW2 SW_Push_4pin, SW3 SW_Push_4pin, SW4 SW_Push_4pin, SW5 SW_Push_4pin, SW6 SW_Push_4pin, SW7 SW_Push_4pin, SW8 SW_Push_4pin, U1 74HC74, U10 74LVC1G38, U11 74LVC1G00, U12 74HC00, U13 74LVC1G38, U14 74HC02, U15 74LVC1G14, U16 74HC4017, U17 74HC4017, U19 74LVC1GX04, U2 74HCS05, U20 74LVC1G04, U21 NE555D, U22 74LVC1G32, U23 74LVC1G04, U24 MIC5504-3.3YM5, U25 74HC08, U26 74LVC2G132, U27 74HC74, U28 74LVC1G02, U29 74HC74, U3 74LVC1G02, U30 74LVC1G04, U4 74HCS05, U5 74LVC1G38, U6 74LVC2G74, U7 74LVC1G08, U8 74HC74, U9 74HCS05, Y1 Crystal

Commit message: Updated schematics and pcbs
Parts:
- removed C24: 100n, Capacitor_SMD:C_0805_2012Metric_Pad1.18x1.45mm_HandSolder, symbol Device:C
- added C18: 100n, Capacitor_SMD:C_0805_2012Metric_Pad1.18x1.45mm_HandSolder, symbol Device:C
- added D2, D3: LED, LED_SMD:LED_0805_2012Metric_Pad1.15x1.40mm_HandSolder, symbol Device:LED
- added J3, J4: Conn_01x02_Male, Connector_PinHeader_2.54mm:PinHeader_1x02_P2.54mm_Horizontal, symbol Connector:Conn_01x02_Male
- added J5: Conn_01x10_Male, Connector_IDC:IDC-Header_2x05_P2.54mm_Vertical, symbol Connector:Conn_01x10_Male
- added R27, R28: 330, Resistor_SMD:R_0805_2012Metric_Pad1.20x1.40mm_HandSolder, symbol Device:R
- added U18: 74LVC2G04, Package_TO_SOT_SMD:SOT-23-6_Handsoldering, symbol riscv-serial:74LVC2G04
- J2: value Conn_01x04_Female -> Conn_01x03; footprint (none) -> Connector_PinHeader_2.54mm:PinHeader_1x03_P2.54mm_Vertical; symbol Connector:Conn_01x04_Female -> Connector:Conn_01x03_Male
- SW1, SW2, SW3, SW4, SW5, SW6, SW7, SW8: footprint (none) -> riscv-serial:SW_SPST_DTSM-6
Connections:
- net CLK: now also J5.9 (Pin_9), U18.1
- net GND: now also J2.3 (Pin_3), C18.2, J3.2 (Pin_2), J4.2 (Pin_2), J5.1 (Pin_1), J5.10 (Pin_10), J5.6 (Pin_6), J5.8 (Pin_8), U18.2 (GND); no longer J2.2 (Pin_2), J2.4 (Pin_4)
- net VCC: now also C18.1, D2.2 (A), D3.2 (A), U18.5 (VCC)
- net WAKEUP: now also J3.1 (Pin_1)
- net ~{CLK}: now also J5.7 (Pin_7), U18.3
- net ~{RESET}: now also J5.5 (Pin_5)
- net ~{SLEEP}: now also J5.4 (Pin_4)
- net ~{WAIT}: now also J4.1 (Pin_1)
- net at R24.3: now also J2.2 (Pin_2); no longer J2.3 (Pin_3)
- net OPDONE renamed OP_DONE
- net OP_DONE: now also J5.3 (Pin_3)
- net STEPDONE renamed STEP_DONE
- net STEP_DONE: now also J5.2 (Pin_2)
- new net: D2.1 (K), R27.1
- new net: D3.1 (K), R28.1
- new net: R28.2, U18.6
- new net: R27.2, U18.4

Commit message: Added two LEDs
Parts:
- removed U26: 74LVC2G132, Package_SO:SSOP-8_2.95x2.8mm_P0.65mm, symbol riscv-serial:74LVC2G132
- added C24, C44, C45: 100n, Capacitor_SMD:C_0805_2012Metric_Pad1.18x1.45mm_HandSolder, symbol Device:C
- added D4, D5: LED, LED_SMD:LED_0805_2012Metric_Pad1.15x1.40mm_HandSolder, symbol Device:LED
- added R29, R30: 330, Resistor_SMD:R_0805_2012Metric_Pad1.20x1.40mm_HandSolder, symbol Device:R
- added U26, U31: 74LVC1G132, Package_TO_SOT_SMD:SOT-23-5_HandSoldering, symbol riscv-serial:74LVC1G132
- added U32, U33: 74LVC1G04, Package_TO_SOT_SMD:SOT-23-5_HandSoldering, symbol riscv-serial:74LVC1G04
- J3, J4: footprint Connector_PinHeader_2.54mm:PinHeader_1x02_P2.54mm_Horizontal -> Connector_PinHeader_2.54mm:PinHeader_1x02_P2.54mm_Vertical
Connections:
- net B_555: now also SW8.1, SW8.2; no longer SW8.3
- net B_OSC: now also SW7.1, SW7.2; no longer SW7.3
- net B_RESET: now also SW6.3
- net GND: now also SW6.2, SW7.3, SW7.4, SW8.3, SW8.4, C24.2, C44.2, C45.2, U26.3 (GND), U31.3 (GND), U32.3 (GND), U33.3 (GND); no longer SW7.1, SW8.1
- net VCC: now also SW1.3, SW1.4, SW2.3, SW2.4, SW3.3, SW3.4, SW4.3, SW4.4, SW5.3, SW5.4, C24.1, C44.1, C45.1, D4.2 (A), D5.2 (A), U26.5 (VCC), U31.5 (VCC), U32.5 (VCC), U33.5 (VCC); no longer SW1.1, SW2.1, SW3.1, SW4.1, SW5.1
- net at R12.2, R13.1: now also SW3.1, SW3.2; no longer SW3.3
- net at R14.2, R15.1: now also SW4.1, SW4.2; no longer SW4.3
- net at C42.1, R23.1: now also U26.1
- net at U25.2: now also U26.2, U31.4
- net at U25.9: now also U26.4, U31.2
- net at SW2.2: now also R8.2, R9.1, SW2.1
- net at R16.2, R17.1: now also SW5.1, SW5.2; no longer SW5.3
- net at SW1.2: now also R6.2, R7.1, SW1.1
- net at C43.1, R26.1: now also U31.1
- net at U25.4, U27.9 (Q): now also U32.2
- net at U25.12, U29.5 (Q): now also U33.2
- new net: R29.2, U32.4
- new net: R30.2, U33.4
- new net LED_555: D5.1 (K), R30.1
- new net LED_OSC: D4.1 (K), R29.1
- no-connect marks 40 -> 24
Other:
- moved on the sheet: C36, C42, C43, D1, D2, D3, J2, J3, J4, J5, R10, R11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
